Commit message: add moveit controls

File: robotic_arm_description/urdf/robotic_arm.xacro (robot description, xacro)
@@ -8,5 +8,5 @@
     <parent link="world"/>
     <child link="base_link"/>
-    <origin rpy="0 0 0" xyz="0.0 0.0 0.00"/>
+    <origin rpy="0 0 ${radians(180)}" xyz="0.0 0.0 0.00"/>
 </joint>
 <link name="base_link">
@@ -190,5 +190,5 @@
   </collision>
 </link>
-<joint name="Revolute 12" type="revolute">
+<joint name="Revolute_12" type="revolute">
   <origin xyz="0.000534 0.058358 0.084193" rpy="0 0 0"/>
   <parent link="base_link"/>
@@ -197,5 +197,5 @@
   <limit upper="6.283185" lower="0.0" effort="100" velocity="100"/>
 </joint>
-<joint name="Revolute 13" type="revolute">
+<joint name="Revolute_13" type="revolute">
   <origin xyz="-0.15 0.02 0.16" rpy="0 0 0"/>
   <parent link="jaw1_1"/>
@@ -204,5 +204,5 @@
   <limit upper="1.570796" lower="-1.047198" effort="100" velocity="100"/>
 </joint>
-<joint name="Revolute 14" type="revolute">
+<joint name="Revolute_14" type="revolute">
   <origin xyz="0.0 0.0 0.35" rpy="0 0 0"/>
   <parent link="jaw2_1"/>
@@ -211,5 +211,5 @@
   <limit upper="3.141593" lower="-0.523599" effort="100" velocity="100"/>
 </joint>
-<joint name="Revolute 15" type="revolute">
+<joint name="Revolute_15" type="revolute">
   <origin xyz="-0.246263 -0.048 0.044252" rpy="0 0 0"/>
   <parent link="jaw3_1"/>
@@ -218,5 +218,5 @@
   <limit upper="3.141593" lower="0.0" effort="100" velocity="100"/>
 </joint>
-<joint name="Revolute 16" type="revolute">
+<joint name="Revolute_16" type="revolute">
   <origin xyz="-0.115 0.0125 0.0" rpy="0 0 0"/>
   <parent link="jaw4_1"/>
@@ -225,5 +225,5 @@
   <limit upper="1.745329" lower="-1.745329" effort="100" velocity="100"/>
 </joint>
-<joint name="Revolute 17" type="revolute">
+<joint name="Revolute_17" type="revolute">
   <origin xyz="-0.093 -0.012 0.0" rpy="0 0 0"/>
   <parent link="jaw5_1"/>
@@ -232,5 +232,5 @@
   <limit upper="3.141593" lower="0.0" effort="100" velocity="100"/>
 </joint>
-<joint name="Revolute 22" type="revolute">
+<joint name="Revolute_22" type="revolute">
   <origin xyz="-0.032892 0.03931 0.009" rpy="0 0 0"/>
   <parent link="jaw6_1"/>
@@ -239,10 +239,10 @@
   <limit upper="0.292343" lower="-1.570796" effort="100" velocity="100"/>
 </joint>
-<joint name="Revolute 24" type="revolute">
+<joint name="Revolute_24" type="revolute">
   <origin xyz="-0.032892 -0.039309 0.009" rpy="0 0 0"/>
   <parent link="jaw6_1"/>
   <child link="jaw7.2_1"/>
   <axis xyz="-0.0 0.0 1.0"/>
-  <limit upper="1.570796" lower="-0.292343" effort="100" velocity="100"/>
+  <limit lower="-0.292343"  upper="1.570796"  effort="100" velocity="100"/>
 </joint>
 </robot>
